Commit message: add depth cam at pineapple urdf

File: pineapple/urdf/pineappleurdf.urdf (robot description, URDF)
Before this commit: robot pineapple, 9 links, 8 joints
Links:
- added link depth_cam, mass 0.30000000; visual mesh filename=../meshes/depth_cam.STL
- link L_calf: mass 0.65000000 -> 0.50000000
- link L_hip: mass 0.64000000 -> 0.57300000
- link L_thigh: mass 0.88000000 -> 0.75000000
- link R_calf: mass 0.65000000 -> 0.50000000
- link R_hip: mass 0.64000000 -> 0.57300000
- link R_thigh: mass 0.88000000 -> 0.75000000
- link base_link: mass 2.65000000 -> 2.85000000
Joints:
- added joint depth_cam_joint: type fixed, parent base_link, child depth_cam, origin xyz=0.134942648598871 0 0.120596007530399 rpy=0 0.698131700797732 0, axis 0 0 0
- joint L_calf_joint: limit lower=-3.3 upper=0 effort=23.7 velocity=30.1 -> lower=-3.1416 upper=0.0 effort=33.5 velocity=21.0
- joint L_hip_joint: limit (none) -> lower=-0.52358 upper=0.17444 effort=23.7 velocity=30.0
- joint L_thigh_joint: limit lower=0 upper=2.1 effort=23.7 velocity=30.1 -> lower=0.0 upper=1.571 effort=23.7 velocity=30.0
- joint L_wheel_joint: limit (none) -> effort=3.69 velocity=60.0; type continuous -> revolute
- joint R_calf_joint: limit lower=-3.3 upper=0 effort=23.7 velocity=30.1 -> lower=-3.1416 upper=0.0 effort=33.5 velocity=21.0
- joint R_hip_joint: limit (none) -> lower=-0.17444 upper=0.52358 effort=23.7 velocity=30.0
- joint R_thigh_joint: limit lower=0 upper=2.1 effort=23.7 velocity=30.1 -> lower=0.0 upper=1.571 effort=23.7 velocity=30.0
- joint R_wheel_joint: limit (none) -> effort=3.69 velocity=60.0; type continuous -> revolute
